Commit message: support longer gripper

File: Gazebo_arm/urdf/tm700_robot_clean.urdf (robot description, URDF)
Before this commit: robot tm700, 11 links, 10 joints
Links:
- link finger_l_link: geometry collision mesh filename=./meshes/toyo_s68/Teeth.stl scale=0.001 0.001 0.001; visual mesh filename=./meshes/toyo_s68/Teeth.stl scale=0.001 0.001 0.001
- link finger_r_link: geometry collision mesh filename=./meshes/toyo_s68/Teeth.stl scale=0.001 0.001 0.001; visual mesh filename=./meshes/toyo_s68/Teeth.stl scale=0.001 0.001 0.001
- link gripper_link: geometry collision mesh filename=./meshes/toyo_s68/Head.stl scale=0.001 0.001 0.001; visual mesh filename=./meshes/toyo_s68/Head.stl scale=0.001 0.001 0.001
- link tip_link: geometry collision box size=0.02 0.02 0.02
Joints:
- joint finger_l_joint: axis 1 0 0 -> 0 -1 0; origin xyz=0.0105 0.0015 0.013 rpy=0 0 0 -> xyz=0.055 0 0.09 rpy=0 0 -1.5707963269
- joint finger_r_joint: axis 1 0 0 -> 0 1 0; origin xyz=-0.0105 0.0015 0.013 rpy=0 0 0 -> xyz=-0.055 0 0.09 rpy=0 0 1.5707963269
- joint gripper_joint: origin xyz=0 0 0.15 rpy=0 0 0 -> xyz=0 0 0.06 rpy=0 0 0

Commit message: add transform for grasping algorithms

File: Gazebo_arm/urdf/tm700_robot_clean.urdf (robot description, URDF)
Before this commit: robot tm700, 11 links, 10 joints
Links:
- added link gripper_b_link
Joints:
- added joint gripper_b_joint: type fixed, parent gripper_link, child gripper_b_link, origin xyz=0 0 0.09 rpy=-1.5707963269 -1.5707963269 0

Commit message: add real grasp algo

File: Gazebo_arm/urdf/tm700_robot_clean.urdf (robot description, URDF)
Before this commit: robot tm700, 12 links, 11 joints
Links:
- added link forbidden_box, mass 0; collision box size=2 2 1; visual box size=2 2 1
Joints:
- added joint forbidden_joint: type fixed, parent forbidden_box, child base_link, origin xyz=0 0 0 rpy=0 0 0

Commit message: a

File: Gazebo_arm/urdf/tm700_robot_clean.urdf (robot description, URDF)
Before this commit: robot tm700, 13 links, 12 joints
Links:
- link gripper_link: geometry 

Commit message: test

File: Gazebo_arm/urdf/tm700_robot_clean.urdf (robot description, URDF)
Before this commit: robot tm700, 13 links, 12 joints
Links:
- link gripper_link: geometry collision mesh filename=./meshes/toyo_s68/Head.stl scale=0.001 0.001 0.001; visual mesh filename=./meshes/toyo_s68/Head.stl scale=0.001 0.001 0.001

Commit message: test GDN with flying gripper

File: Gazebo_arm/urdf/tm700_robot_clean.urdf (robot description, URDF)
Before this commit: robot tm700, 13 links, 12 joints
Links:
- link tip_link: geometry collision box size=0.02 0.02 0.02; visual box size=0.02 0.02 0.02
Joints:
- joint gripper_b_joint: origin xyz=0 0 0.09 rpy=-1.5707963269 -1.5707963269 0 -> xyz=0 0 0.095 rpy=-1.5707963269 -1.5707963269 0
